Commit message: Adding solutions

File: src/bar_examples/my_first_robot/robot_description/first_robot.urdf.xacro (robot description, xacro)
@@ -1,5 +1,5 @@
 <?xml version='1.0' encoding='utf-8'?>
 <robot xmlns:xacro="http://www.ros.org/wiki/xacro" name="krytn">
-    <xacro:include filename="$(find my_first_robot_freecad)/urdf/FirstRobot.urdf" />
+    <xacro:include filename="$(find forklift_freecad)/urdf/FirstRobot.urdf" />
     <gazebo reference="caster_wheel">
         <collision>
@@ -73,4 +73,31 @@
             <state_interface name="effort" />
         </joint>
+        <joint name="back_right_joint">
+            <command_interface name="velocity">
+                <param name="min">-10</param>
+                <param name="max">10</param>
+            </command_interface>
+            <state_interface name="position"/>
+            <state_interface name="velocity"/>
+            <state_interface name="effort" />
+        </joint>
+        <joint name="back_left_joint">
+            <command_interface name="velocity">
+                <param name="min">-10</param>
+                <param name="max">10</param>
+            </command_interface>
+            <state_interface name="position"/>
+            <state_interface name="velocity"/>
+            <state_interface name="effort" />
+        </joint>
+        <joint name="tines_joint">
+            <command_interface name="velocity">
+                <param name="min">-10</param>
+                <param name="max">10</param>
+            </command_interface>
+            <state_interface name="position"/>
+            <state_interface name="velocity"/>
+            <state_interface name="effort" />
+        </joint>
     </ros2_control>
     <!-- Setup Gazebo plugins -->

Commit message: Addding sensors

File: src/bar_examples/my_first_robot/robot_description/first_robot.urdf.xacro (robot description, xacro)
@@ -1,5 +1,14 @@
 <?xml version='1.0' encoding='utf-8'?>
 <robot xmlns:xacro="http://www.ros.org/wiki/xacro" name="krytn">
+    <xacro:include filename="$(find magni_description)/urdf/inertial.xacro" />
     <xacro:include filename="$(find forklift_freecad)/urdf/FirstRobot.urdf" />
+    <xacro:include filename="$(find sensors)/realsense_d435/realsense.urdf.xacro" />
+    <xacro:include filename="$(find sensors)/lidar_2d/lidar_2d.urdf.xacro" />
+    <xacro:realsense world_link_name="base_link">
+        <origin xyz="-0.7 0 2.4" rpy="0 0 ${pi}" />
+    </xacro:realsense>
+    <xacro:lidar_2d world_link_name="base_link">
+        <origin xyz="-0.4 0 1.1" rpy="0 0 0" />
+    </xacro:lidar_2d>
     <gazebo reference="caster_wheel">
         <collision>

Commit message: Final code adjustments

File: src/bar_examples/my_first_robot/robot_description/first_robot.urdf.xacro (robot description, xacro)
@@ -5,4 +5,10 @@
     <xacro:include filename="$(find sensors)/realsense_d435/realsense.urdf.xacro" />
     <xacro:include filename="$(find sensors)/lidar_2d/lidar_2d.urdf.xacro" />
+    <link name="base_footprint" />
+    <joint name="base_footprint_joint" type="fixed">
+        <parent link="base_footprint" />
+        <child link="base_link" />
+        <origin rpy="0 0 ${pi}" />
+    </joint>
     <xacro:realsense world_link_name="base_link">
         <origin xyz="-0.7 0 2.4" rpy="0 0 ${pi}" />
@@ -101,5 +107,5 @@
         </joint>
         <joint name="tines_joint">
-            <command_interface name="velocity">
+            <command_interface name="position">
                 <param name="min">-10</param>
                 <param name="max">10</param>

File: src/bar_examples/sensors/lidar_2d/lidar_2d.urdf.xacro (robot description, xacro)
@@ -30,13 +30,13 @@
                     <scan>
                         <horizontal>
-                            <samples>180</samples>
+                            <samples>360</samples>
                             <resolution>1</resolution>
-                            <min_angle>-2.356195</min_angle>
-                            <max_angle>2.356195</max_angle>
+                            <min_angle>-3.14</min_angle>
+                            <max_angle>3.14</max_angle>
                         </horizontal>
                     </scan>
                     <range>
-                        <min>0.060</min>
-                        <max>5</max>
+                        <min>0.40</min>
+                        <max>30</max>
                         <resolution>0.01</resolution>
                     </range>

File: src/forklift_freecad/urdf/FirstRobot.urdf (robot description, URDF)
Before this commit: robot Robot, 6 links, 5 joints
Links:
- link back_left_wheel: geometry collision cylinder length=0.1000000000000005 radius=0.1; visual mesh filename=package://forklift_freecad/meshes/forkliftv2_Body.dae
- link back_right_wheel: geometry collision cylinder length=0.1000000000000005 radius=0.1; visual mesh filename=package://forklift_freecad/meshes/forkliftv2_Body.dae
- link base_link: mass 200.4799999999999995 -> 100.0; geometry collision mesh filename=package://forklift_freecad/meshes/forkliftv2_Forklift_Chass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; visual mesh filename=package://forklift_freecad/meshes/forkliftv2_Forklift_Chass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
- link left_wheel: geometry collision cylinder length=0.03000000000000005 radius=0.1; visual mesh filename=package://forklift_freecad/meshes/forkliftv2_Body.dae
- link right_wheel: geometry collision cylinder length=0.1000000000000005 radius=0.1; visual mesh filename=package://forklift_freecad/meshes/forkliftv2_Body.dae
- link tines_link: geometry collision mesh filename=package://forklift_freecad/meshes/forkliftv2_Body002.dae; visual mesh filename=package://forklift_freecad/meshes/forkliftv2_Body002.dae
Joints:
- joint back_left_joint: origin xyz=-0.3 -0.5 0.0 rpy=-1.5707963267948966 0.0 0.0 -> xyz=-0.3 -0.3 0.0 rpy=-1.5707963267948966 0.0 0.0
- joint back_right_joint: origin xyz=-0.3 0.5 0.0 rpy=-1.5707963267948966 0.0 0.0 -> xyz=-0.3 0.3 0.0 rpy=-1.5707963267948966 0.0 0.0
- joint left_wheel_joint: origin xyz=-0.8 0.5 0.0 rpy=-1.5707963267948966 0.0 0.0 -> xyz=-0.8 -0.3 0.0 rpy=-1.5707963267948966 0.0 0.0
- joint right_wheel_joint: origin xyz=-0.8 -0.5 0.0 rpy=-1.5707963267948966 0.0 0.0 -> xyz=-0.8 0.3 0.0 rpy=-1.5707963267948966 0.0 0.0
- joint tines_joint: limit lower=0.0 upper=1.0 effort=1.0 velocity=1.0 -> lower=-0.1 upper=1.0 effort=10000.0 velocity=10.0; origin xyz=0.0 0.75 0.0 rpy=0.0 -0.0 0.0 -> xyz=-0.0 0.0 0.0 rpy=0.0 -0.0 0.0
