Commit message: Playing with ideas for automated detection

File: src/bar_examples/sensors/realsense_d435/realsense.urdf.xacro (robot description, xacro)
@@ -1,6 +1,6 @@
 <robot name="sensor_d435"
     xmlns:xacro="http://ros.org/wiki/xacro">
-    <xacro:macro name="realsense" params="world_link_name *origin">
-        <link name="realsense_link">
+    <xacro:macro name="realsense" params="world_link_name prefix:='' *origin">
+        <link name="${prefix}realsense_link">
             <xacro:box_inertial x="0.02" y="0.1" z="0.01" mass="0.06"/>
             <collision name="collision">
@@ -37,10 +37,10 @@
             </visual>
         </link>
-        <gazebo reference="realsense_link">
-            <sensor name="realsense_d435" type="rgbd_camera">
+        <gazebo reference="${prefix}realsense_link">
+            <sensor name="${prefix}realsense_d435" type="rgbd_camera">
                 <update_rate>10</update_rate>
-                <topic>realsense</topic>
+                <topic>${prefix}realsense</topic>
                 <camera name="camera">
-                    <optical_frame_id>realsense</optical_frame_id>
+                    <optical_frame_id>${prefix}realsense</optical_frame_id>
                     <horizontal_fov>1.0472</horizontal_fov>
                     <image>
@@ -56,6 +56,6 @@
             </sensor>
         </gazebo>
-        <joint name="realsense_joint" type="fixed">
-            <child link="realsense_link" />
+        <joint name="${prefix}realsense_joint" type="fixed">
+            <child link="${prefix}realsense_link" />
             <parent link="${world_link_name}" />
             <xacro:insert_block name="origin"/>

File: src/my_robot_arm/urdf/my_robot_arm.urdf.xacro (robot description, xacro)
@@ -10,7 +10,4 @@
     </xacro:ur_robot>
     <link name="world" />
-    <xacro:realsense world_link_name="world">
-        <origin xyz="0 2.00 2.2" rpy="0 ${pi/4} -${pi/2}" />
-    </xacro:realsense>
     <link name="base_link">
         <visual>
@@ -124,3 +121,8 @@
         </plugin>
     </gazebo>
+    <!--
+    <xacro:realsense world_link_name="world" prefix="close_up_">
+        <origin xyz="-0.5 -0.5 -0.5" rpy="0 0 ${pi/4}" />
+    </xacro:realsense>
+    -->
 </robot>

Commit message: experimenting with vision. Figured out how to get the octomap to work closer

File: src/bar_examples/sensors/realsense_d435/realsense.urdf.xacro (robot description, xacro)
@@ -7,5 +7,5 @@
                 <origin rpy="0 0 ${pi/2}"/>
                 <geometry>
-                    <mesh filename="package://sensors/realsense_d435/meshes/realsense.dae" />
+                    <box size="0.2 0.2 0.2" />
                 </geometry>
             </collision>
@@ -39,5 +39,5 @@
         <gazebo reference="${prefix}realsense_link">
             <sensor name="${prefix}realsense_d435" type="rgbd_camera">
-                <update_rate>10</update_rate>
+                <update_rate>2</update_rate>
                 <topic>${prefix}realsense</topic>
                 <camera name="camera">
@@ -51,5 +51,5 @@
                     <clip>
                         <near>0.01</near>
-                        <far>300</far>
+                        <far>5</far>
                     </clip>
                 </camera>

File: src/my_robot_arm/urdf/my_robot_arm.urdf.xacro (robot description, xacro)
@@ -3,4 +3,7 @@
     <xacro:include filename="$(find magni_description)/urdf/inertial.xacro" />
     <xacro:include filename="$(find sensors)/realsense_d435/realsense.urdf.xacro" />
+    <xacro:realsense world_link_name="ur5_base">
+        <origin xyz="0 0.2 -0.6" rpy="0 -${pi/2} -${pi/2}" />
+    </xacro:realsense>
     <!-- Include a UR5 -->
     <xacro:include filename="$(find ur_description)/urdf/ur_macro.xacro" />
