Commit message: Getting the full pipeline working

File: src/my_robot_arm/urdf/my_robot_arm.urdf.xacro (robot description, xacro)
@@ -4,5 +4,5 @@
     <xacro:include filename="$(find sensors)/realsense_d435/realsense.urdf.xacro" />
     <xacro:realsense world_link_name="ur5_base">
-        <origin xyz="0 0.2 -0.6" rpy="0 -${pi/2} -${pi/2}" />
+        <origin xyz="0 0.0 0.6" rpy="${pi} 0 ${3*pi/4}" />
     </xacro:realsense>
     <!-- Include a UR5 -->
@@ -56,5 +56,5 @@
         <origin rpy="0.0 -0.0 0.0" xyz="-0.06 0.001 0.06"/>
         <axis xyz="1 0 0"/>
-        <limit effort="1000.0" lower="-0.1" upper="0.078" velocity="1000.1"/>
+        <limit effort="1000.0" lower="-0.01" upper="0.078" velocity="1000.1"/>
     </joint>
     <joint name="gripper_joint" type="fixed">
